File: vfobox.sch (EAGLE design)
At the start: 36 parts, among them IC1 78L05F, Q1 2N3904, Q2 2N3904, SW1 ROTARTY_ENCODER, U1 LCD-16X2SILK, U2 ATMEGA328P_PDIP

Commit message: revised schematic
Parts:
- added R11, R13: 4k7, SparkFun-Passives:RESISTORKIT
- D2: value (none) -> 1N34
- L1: value (none) -> 3.3uH
- R1: value 4k7 -> 10k
Connections:
- new net N$19: R11.2, R13.2, R2.2
- net +5V: no longer R2.2
- net SCL: now also R13.1
- net SDA: now also R11.1
Other:
- note removed: "(no pullups)"
- moved on the sheet: C4, R2, R3, R4
